Commit message: created mjcf with proper limits

File: friday_description/friday.urdf (robot description, URDF)
Before this commit: robot friday_robot, 18 links, 17 joints
Links:
- removed link virtual_link
- link base_link: geometry collision mesh filename=package://champ_description/meshes/base_link.STL; visual mesh filename=package://champ_description/meshes/base_link.STL
- link fl_abad_link: geometry collision mesh filename=package://champ_description/meshes/fl_abad_link.STL; visual mesh filename=package://champ_description/meshes/fl_abad_link.STL
- link fl_foot_link: geometry collision mesh filename=package://champ_description/meshes/fl_foot_link.STL; visual mesh filename=package://champ_description/meshes/fl_foot_link.STL
- link fl_lower_leg_link: geometry collision mesh filename=package://champ_description/meshes/fl_lower_leg_link.STL; visual mesh filename=package://champ_description/meshes/fl_lower_leg_link.STL
- link fl_upper_leg_link: geometry collision mesh filename=package://champ_description/meshes/fl_upper_leg_link.STL; visual mesh filename=package://champ_description/meshes/fl_upper_leg_link.STL
- link fr_abad_link: geometry collision mesh filename=package://champ_description/meshes/fr_abad_link.STL; visual mesh filename=package://champ_description/meshes/fr_abad_link.STL
- link fr_foot_link: geometry collision mesh filename=package://champ_description/meshes/fr_foot_link.STL; visual mesh filename=package://champ_description/meshes/fr_foot_link.STL
- link fr_lower_leg_link: geometry collision mesh filename=package://champ_description/meshes/fr_lower_leg_link.STL; visual mesh filename=package://champ_description/meshes/fr_lower_leg_link.STL
- link fr_upper_leg_linnk: geometry collision mesh filename=package://champ_description/meshes/fr_upper_leg_linnk.STL; visual mesh filename=package://champ_description/meshes/fr_upper_leg_linnk.STL
- link hl_abad_link: geometry collision mesh filename=package://champ_description/meshes/hl_abad_link.STL; visual mesh filename=package://champ_description/meshes/hl_abad_link.STL
- link hl_foot_link: geometry collision mesh filename=package://champ_description/meshes/hl_foot_link.STL; visual mesh filename=package://champ_description/meshes/hl_foot_link.STL
- link hl_lower_leg_link: geometry collision mesh filename=package://champ_description/meshes/hl_lower_leg_link.STL; visual mesh filename=package://champ_description/meshes/hl_lower_leg_link.STL
- link hl_upper_leg_linnk: geometry collision mesh filename=package://champ_description/meshes/hl_upper_leg_linnk.STL; visual mesh filename=package://champ_description/meshes/hl_upper_leg_linnk.STL
- link hr_abad_link: geometry collision mesh filename=package://champ_description/meshes/hr_abad_link.STL; visual mesh filename=package://champ_description/meshes/hr_abad_link.STL
- link hr_foot_link: geometry collision mesh filename=package://champ_description/meshes/hr_foot_link.STL; visual mesh filename=package://champ_description/meshes/hr_foot_link.STL
- link hr_lower_leg_link: geometry collision mesh filename=package://champ_description/meshes/hr_lower_leg_link.STL; visual mesh filename=package://champ_description/meshes/hr_lower_leg_link.STL
- link hr_upper_leg_link: geometry collision mesh filename=package://champ_description/meshes/hr_upper_leg_link.STL; visual mesh filename=package://champ_description/meshes/hr_upper_leg_link.STL
Joints:
- removed joint virtual_joint
- joint fl_abad_joint: limit lower=-1.5 upper=1.5 effort=0 velocity=0 -> lower=-0.67 upper=0.85 effort=0 velocity=0
- joint fl_hip_joint: limit lower=-1.5 upper=1.5 effort=0 velocity=0 -> lower=-1.75 upper=1.75 effort=0 velocity=0
- joint fl_knee_joint: limit lower=-1.5 upper=1.5 effort=0 velocity=0 -> lower=-3.14 upper=0.0 effort=0 velocity=0
- joint fr_abad_joint: limit lower=-1.5 upper=1.5 effort=0 velocity=0 -> lower=-0.85 upper=0.67 effort=0 velocity=0
- joint fr_hip_joint: limit lower=-1.5 upper=1.5 effort=0 velocity=0 -> lower=-1.75 upper=1.75 effort=0 velocity=0
- joint fr_knee_joint: limit lower=-1.5 upper=1.5 effort=0 velocity=0 -> lower=-3.14 upper=0.0 effort=0 velocity=0
- joint hl_abad_joint: limit lower=-1.5 upper=1.5 effort=0 velocity=0 -> lower=-0.67 upper=0.85 effort=0 velocity=0
- joint hl_hip_joint: limit lower=-1.5 upper=1.5 effort=0 velocity=0 -> lower=-1.75 upper=1.75 effort=0 velocity=0
- joint hl_knee_joint: limit lower=-1.5 upper=1.5 effort=0 velocity=0 -> lower=-3.14 upper=0.0 effort=0 velocity=0
- joint hr_abad_joint: limit lower=-1.5 upper=1.5 effort=0 velocity=0 -> lower=-0.85 upper=0.67 effort=0 velocity=0
- joint hr_hip_joint: limit lower=-1.5 upper=1.5 effort=0 velocity=0 -> lower=-1.75 upper=1.75 effort=0 velocity=0
- joint hr_knee_joint: limit lower=-1.5 upper=1.5 effort=0 velocity=0 -> lower=-3.14 upper=0.0 effort=0 velocity=0

File: src/champ/champ_description/urdf/friday.urdf (robot description, URDF)
Before this commit: robot friday, 17 links, 16 joints
Joints:
- joint fl_abad_joint: limit lower=-1.5 upper=1.5 effort=0 velocity=0 -> lower=-0.67 upper=0.85 effort=0 velocity=0
- joint fl_hip_joint: limit lower=-1.5 upper=1.5 effort=0 velocity=0 -> lower=-1.75 upper=1.75 effort=0 velocity=0
- joint fl_knee_joint: limit lower=-1.5 upper=1.5 effort=0 velocity=0 -> lower=-3.14 upper=0.0 effort=0 velocity=0
- joint fr_abad_joint: limit lower=-1.5 upper=1.5 effort=0 velocity=0 -> lower=-0.85 upper=0.67 effort=0 velocity=0
- joint fr_hip_joint: limit lower=-1.5 upper=1.5 effort=0 velocity=0 -> lower=-1.75 upper=1.75 effort=0 velocity=0
- joint fr_knee_joint: limit lower=-1.5 upper=1.5 effort=0 velocity=0 -> lower=-3.14 upper=0.0 effort=0 velocity=0
- joint hl_abad_joint: limit lower=-1.5 upper=1.5 effort=0 velocity=0 -> lower=-0.67 upper=0.85 effort=0 velocity=0
- joint hl_hip_joint: limit lower=-1.5 upper=1.5 effort=0 velocity=0 -> lower=-1.75 upper=1.75 effort=0 velocity=0
- joint hl_knee_joint: limit lower=-1.5 upper=1.5 effort=0 velocity=0 -> lower=-3.14 upper=0.0 effort=0 velocity=0
- joint hr_abad_joint: limit lower=-1.5 upper=1.5 effort=0 velocity=0 -> lower=-0.85 upper=0.67 effort=0 velocity=0
- joint hr_hip_joint: limit lower=-1.5 upper=1.5 effort=0 velocity=0 -> lower=-1.75 upper=1.75 effort=0 velocity=0
- joint hr_knee_joint: limit lower=-1.5 upper=1.5 effort=0 velocity=0 -> lower=-3.14 upper=0.0 effort=0 velocity=0
